File: canhat.kicad_pcb (KiCad board)
At the start: 2 copper layers, 65 x 30 mm, 41 parts, among them J1 Raspberry_Pi_2_3, J2 CAN In/Out/GND, J3 GPIO, J5 12V, U1 MCP2515-xSO, U2 SN65HVDA541, U3 AT24C32-SSHM, U4 AP63205, Y1 16MHz

Commit message: First Commit
Parts:
- removed OSHW1: Logo_Open_Hardware_Small, Symbol:OSHW-Logo_5.7x6mm_SilkScreen
Connections:
- net /~CS renamed /~{CS}
- net /~INT renamed /~{INT}
Other:
- net class CAN removed
- net class Default removed
- net class Power removed
